File: CLOCKS.kicad_sch (KiCad schematic)
At the start: 0 parts

Commit message: Worked a bit more on CLOCKS.kicad_sch.
Parts:
- added C10: 10uF, symbol Device:C_Small
- added C11: 1uF, Capacitor_SMD:C_0402_1005Metric, symbol Device:C_Small
- added C12: 100nF, Capacitor_SMD:C_0201_0603Metric, symbol Device:C_Small
- added C25: 10nf, Capacitor_SMD:C_0201_0603Metric, symbol Device:C_Small
- added FB1: 220@100 MHz, Inductor_SMD:L_Bourns_SRP1038C_10.0x10.0mm, symbol Device:FerriteBead_Small
- added IC1: LMK04828BISQ_NOPB, QFN50P900X900X80-65N, symbol SamacSys_Parts:LMK04828BISQ_NOPB
- added R28: 22, Resistor_SMD:R_0402_1005Metric, symbol Device:R_Small
- added R29, R30: 10K, Resistor_SMD:R_0402_1005Metric, symbol Device:R_Small
- added TP7: CLK 100MHZ, TestPoint:TestPoint_Pad_D2.0mm, symbol Connector:TestPoint
- added TP8: PRE RES CLK, TestPoint:TestPoint_Pad_D2.0mm, symbol Connector:TestPoint
- added Y1: AOCJY1A-100.000MHZ-E, AOCJY1A-100.000MHZ-E:XTAL_AOCJY1A-100.000MHZ-E, symbol AOCJY1A-100.000MHZ-E:AOCJY1A-100.000MHZ-E
Connections:
- new net: R28.1, TP8.1, Y1.8 (OUTPUT)
- new net: C25.2, R29.1, R30.2, Y1.1 (VC)
- new net: C10.1, C11.1, C12.1, FB1.1, Y1.14 (VDD)
- new net 5V: FB1.2, R29.2
- new net CLK_100MHZ_REF: R28.2, TP7.1
- new net GND: C10.2, C11.2, C12.2, C25.1, R30.1, Y1.7 (GND)

Commit message: Added net names to CLOCKS.kicad_sch.
Parts:
- added C26, C27, C28, C29, C30, C31, C32, C5, C6, C7, C8, C9: 100nF, Capacitor_SMD:C_0201_0603Metric, symbol Device:C_Small
- C10: footprint (none) -> Resistor_SMD:R_0603_1608Metric
Connections:
- net GND: now also C26.1, C27.1, C28.1, C29.1, C31.1, C32.2, C5.2, C6.2, C7.1, C8.1, C9.1
- net DCLKOUT0_1: now reaches IC1.1 (DCLKOUT0_1)
- net 3v3: now reaches IC1.10 (VCC1_VCO)
- net 3v3: now also IC1.17 (VCC2_CG1), IC1.21 (VCC3_SYSREF), IC1.26 (VCC4_CG2), IC1.33 (VCC5_DIG), IC1.36 (VCC6_PLL1), IC1.39 (VCC7_OSCOUT), IC1.42 (VCC8_OSCIN), IC1.45 (VCC9_CP2), IC1.47 (VCC10_PLL2), IC1.53 (VCC11_CG3), IC1.64 (VCC12_CG0), C26.2, C27.2, C28.2, C29.2, C30.2, C31.2, C32.1, C5.1, C6.1, C7.2, C8.2, C9.2
- net LDOBYP1: now reaches IC1.11 (LDOBYP1)
- net LDOBYP2: now reaches IC1.12 (LDOBYP2)
- net SDCLKOUT3_1: now reaches IC1.13 (SDCLKOUT3_1)
- net SDCLKOUT3_2: now reaches IC1.14 (SDCLKOUT3_2)
- net DCLKOUT2_1: now reaches IC1.15 (DCLKOUT2_1)
- net DCLKPOUT2_2: now reaches IC1.16 (DCLKOUT2_2)
- net LMK0482 CS: now reaches IC1.18 (CS)
- net LMK04828 SCK: now reaches IC1.19 (SCK)
- net DCLKOUT0_2: now reaches IC1.2 (DCLKOUT0_2)
- net LMK04828 SDIO: now reaches IC1.20 (SDIO)
- net SDCLKOUT5_1: now reaches IC1.22 (SDCLKOUT5_1)
- net SDCLKOUT5_2: now reaches IC1.23 (SDCLKOUT5_2)
- net DCLKOUT4_1: now reaches IC1.24 (DCLKOUT4_1)
- net DCLKOUT4_2: now reaches IC1.25 (DCLKOUT4_2)
- net DCLKOUT6_1: now reaches IC1.27 (DCLKOUT6_1)
- net DCLKOUT6_2: now reaches IC1.28 (DCLKOUT6_2)
- net SDCLKOUT7_1: now reaches IC1.29 (SDCLKOUT7_1)
- net SDCLKOUT1_1: now reaches IC1.3 (SDCLKOUT1_1)
- net SDCLKOUT7_2: now reaches IC1.30 (SDCLKOUT7_2)
- net STATUS_LD1: now reaches IC1.31 (STATUS_LD1)
- net CPOUT1: now reaches IC1.32 (CPOUT1)
- net CLKIN1/FIN/FBCLKIN_1: now reaches IC1.34 (CLKIN1/FIN/FBCLKIN_1)
- net CLKIN1/FIN/FBCLKIN_2: now reaches IC1.35 (CLKIN1/FIN/FBCLKIN_2)
- net CLKIN0_1: now reaches IC1.37 (CLKIN0_1)
- net CLKIN0_2: now reaches IC1.38 (CLKIN0_2)
- net SDCLKOUT1_2: now reaches IC1.4 (SDCLKOUT1_2)
- net OSCOUT/CLKIN2_1: now reaches IC1.40 (OSCOUT/CLKIN2_1)
- net OSCOUT/CLKIN2_2: now reaches IC1.41 (OSCOUT/CLKIN2_2)
- net OSCIN_1: now reaches IC1.43 (OSCIN_1)
- net OSCIN_2: now reaches IC1.44 (OSCIN_2)
- net CPOUT2: now reaches IC1.46 (CPOUT2)
- net STATUS_LD2: now reaches IC1.48 (STATUS_LD2)
- net SDCLKOUT9_1: now reaches IC1.49 (SDCLKOUT9_1)
- net RESET/GPO: now reaches IC1.5 (RESET/GPO)
- net SDCLKOUT9_2: now reaches IC1.50 (SDCLKOUT9_2)
- net DCLKOUT8_1: now reaches IC1.51 (DCLKOUT8_1)
- net DCLKOUT8_2: now reaches IC1.52 (DCLKOUT8_2)
- net DCLKOUT10_1: now reaches IC1.54 (DCLKOUT10_1)
- net DCLKOUT10_2: now reaches IC1.55 (DCLKOUT10_2)
- net SDCLKOUT11_1: now reaches IC1.56 (SDCLKOUT11_1)
- net SDCLKOUT11_2: now reaches IC1.57 (SDCLKOUT11_2)
- net CLKIN_SEL0: now reaches IC1.58 (CLKIN_SEL0)
- net CLKIN_SEL1: now reaches IC1.59 (CLKIN_SEL1)
- net SYNC/SYSREF_REQ: now reaches IC1.6 (SYNC/SYSREF_REQ)
- net SDCLKOUT13_1: now reaches IC1.60 (SDCLKOUT13_1)
- net SDCLKOUT13_2: now reaches IC1.61 (SDCLKOUT13_2)
- net SDCLKOUT12_1: now reaches IC1.62 (DCLKOUT12_1)
- net SDCLKOUT12_2: now reaches IC1.63 (DCLKOUT12_2)
- net DAP: now reaches IC1.65 (DAP)
- net NC_1: now reaches IC1.7 (NC_1)
- net NC_2: now reaches IC1.8 (NC_2)
- net NC_3: now reaches IC1.9 (NC_3)
Other:
- moved on the sheet: IC1
