File: POWER_RAILS.kicad_sch (KiCad schematic)
At the start: 42 parts, among them J4 USB_C_Receptacle, J5 Barrel_Jack_Switch_Pin3Ring, J6 Conn_01x02_Pin, U1 TPS7A9401DSCR, U3 TPS7A9401DSCR, U4 TPS62933PDRLR

Commit message: Added ADC.kicad_sch and CLOCKS.kicad_sch.
Parts:
- added C4: 10pF, Capacitor_SMD:C_0201_0603Metric_Pad0.64x0.40mm_HandSolder, symbol Device:C_Small
- added C5: 4.7uF, Capacitor_SMD:C_0402_1005Metric, symbol Device:C_Small
- added C6: 10pF, Capacitor_SMD:C_0201_0603Metric, symbol Device:C_Small
- added R10: 1467K, Capacitor_SMD:C_0402_1005Metric, symbol Device:R_Small
- added R6: 226k, Resistor_SMD:R_0402_1005Metric, symbol Device:R_Small
- added R7: 100K, Resistor_SMD:R_0402_1005Metric, symbol Device:R_Small
- added R8: 7.32K, Resistor_SMD:R_0201_0603Metric, symbol Device:R_Small
- added R9: 100k, Resistor_SMD:R_0402_1005Metric, symbol Device:R
- added TP1: 1V1, TestPoint:TestPoint_Pad_D1.5mm, symbol Connector:TestPoint
- added TP2: 2v8, TestPoint:TestPoint_Pad_D1.5mm, symbol Connector:TestPoint
- added TP3: 3v3, TestPoint:TestPoint_Pad_D1.5mm, symbol Connector:TestPoint
- added TP4: 5V, TestPoint:TestPoint_Pad_D1.5mm, symbol Connector:TestPoint
- added TP5: Vin, TestPoint:TestPoint_Pad_D1.5mm, symbol Connector:TestPoint
- added U2: TPS7A9401DSCR, TPS7A9401DSCR:VREG_TPS7A9401DSCR, symbol TPS7A9401DSCR:TPS7A9401DSCR
Connections:
- net 2v8: now also TP2.1
- net 3v3: now also TP3.1
- net 5V: now also C4.1, R6.1, TP4.1, U2.1 (IN), U2.2 (IN)
- net GND: now also C4.2, C5.2, C6.2, R7.2, R8.2, R9.1, U2.11 (EXP), U2.4 (PG), U2.6 (GND)
- net Vin: now also TP5.1
- net VBUS: now reaches 3A2.2, C13.2, C14.2, D2.2 (A)
- new net: R10.1, R9.2, U2.5 (FB_PG)
- new net: R6.2, R7.1, U2.3 (EN_UV)
- new net: C5.1, R8.1, U2.7 (NR/SS)
- new net 1V1: C6.1, R10.2, TP1.1, U2.8 (SNS), U2.9 (OUT)
Other:
- company: (none) -> //COLDJOINT
- title: (none) -> ReachSDR
- moved on the sheet: 3A2, C13, C14, D2, J4, R13, R14

Commit message: Worked a bit more on CLOCKS.kicad_sch.
Parts:
- added C7: 10pF, Capacitor_SMD:C_0201_0603Metric_Pad0.64x0.40mm_HandSolder, symbol Device:C_Small
- added C8: 4.7uF, Capacitor_SMD:C_0402_1005Metric, symbol Device:C_Small
- added C9: 10pF, Capacitor_SMD:C_0201_0603Metric, symbol Device:C_Small
- added R11: 226k, Resistor_SMD:R_0402_1005Metric, symbol Device:R_Small
- added R12: 100K, Resistor_SMD:R_0402_1005Metric, symbol Device:R_Small
- added R25: 22.1k, Resistor_SMD:R_0201_0603Metric, symbol Device:R_Small
- added R26: 100k, Resistor_SMD:R_0402_1005Metric, symbol Device:R
- added R27: 1467K, Capacitor_SMD:C_0402_1005Metric, symbol Device:R_Small
- added TP6: 3v3, TestPoint:TestPoint_Pad_D1.5mm, symbol Connector:TestPoint
- added U5: TPS7A9401DSCR, TPS7A9401DSCR:VREG_TPS7A9401DSCR, symbol TPS7A9401DSCR:TPS7A9401DSCR
- DNP2: footprint (none) -> Capacitor_SMD:C_0201_0603Metric
- U4: footprint TPS62933PDRLR:SOFL50P160X60-8N -> TPS62933P:SOFL50P160X60-8N
Connections:
- net 3v3: now also C9.1, R27.2, TP6.1, U5.8 (SNS), U5.9 (OUT)
- net 5V: now also C7.1, R11.1, U5.1 (IN), U5.2 (IN)
- net GND: now also C7.2, C8.2, C9.2, R12.2, R25.2, R26.1, U5.11 (EXP), U5.4 (PG), U5.6 (GND)
- new net: C8.1, R25.1, U5.7 (NR/SS)
- new net: R11.2, R12.1, U5.3 (EN_UV)
- new net: R26.2, R27.1, U5.5 (FB_PG)
Other:
- moved on the sheet: C1, C2, C3, C4, C5, C6, R1, R10, R2, R3, R4, R5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

Commit message: Added net names to CLOCKS.kicad_sch.
Parts:
- removed C5, C8: 4.7uF, Capacitor_SMD:C_0402_1005Metric, symbol Device:C_Small
- removed C6, C9: 10pF, Capacitor_SMD:C_0201_0603Metric, symbol Device:C_Small
- removed C7: 10pF, Capacitor_SMD:C_0201_0603Metric_Pad0.64x0.40mm_HandSolder, symbol Device:C_Small
- removed R10, R27: 1467K, Capacitor_SMD:C_0402_1005Metric, symbol Device:R_Small
- removed R11, R6: 226k, Resistor_SMD:R_0402_1005Metric, symbol Device:R_Small
- removed R12, R7: 100K, Resistor_SMD:R_0402_1005Metric, symbol Device:R_Small
- removed R25: 22.1k, Resistor_SMD:R_0201_0603Metric, symbol Device:R_Small
- removed R26, R4, R9: 100k, Resistor_SMD:R_0402_1005Metric, symbol Device:R
- removed R8: 7.32K, Resistor_SMD:R_0201_0603Metric, symbol Device:R_Small
- removed TP2: 2v8, TestPoint:TestPoint_Pad_D1.5mm, symbol Connector:TestPoint
- removed TP6: 3v3, TestPoint:TestPoint_Pad_D1.5mm, symbol Connector:TestPoint
- removed U2, U5: TPS7A9401DSCR, TPS7A9401DSCR:VREG_TPS7A9401DSCR, symbol TPS7A9401DSCR:TPS7A9401DSCR
- added R4: 100K, Resistor_SMD:R_0402_1005Metric, symbol Device:R_Small
- C4: value 10pF -> 100nF; footprint Capacitor_SMD:C_0201_0603Metric_Pad0.64x0.40mm_HandSolder -> Capacitor_SMD:C_0201_0603Metric
- R3: value 18.7k -> 7.33K
- TP1: value 1V1 -> 1v1
Connections:
- net 2v8 is gone; now on net 1V1: C3.1, R5.2, U1.8 (SNS), U1.9 (OUT)
- net 3v3: now also C4.1
- net 5V: no longer C4.1
- net GND: now also R4.1
- net at R5.1, U1.5 (FB_PG): now also R4.2
Other:
- note added: "TPS7A9401DSCR VOUT = INR/SS(NOM) × RNR/SS"
